File: SEIA-Hardware.kicad_sch (KiCad schematic)
At the start: 3 parts, among them IC1 MIMXRT1062DVL6A, IC2 BMF055, IC3 TLV70433DBVEVM-712

Commit message: added power symbols
Parts:
- added P1: ~, symbol SEIA_SpecLib:BAT
Connections:
- net GND: now also IC3.1 (GND), P1. (GND)
- net +BATT: now reaches IC3.2 (IN)
- net +BATT: now also P1. (GND)
- net +3V3: now reaches IC3.3 (OUT)
- no-connect marks 0 -> 2
Other:
- moved on the sheet: IC3
